File: base/base.kicad_pcb (KiCad board)
At the start: 2 copper layers, 100 x 100 mm, 109 parts, among them J1 Screw_Terminal_01x02, J2 Out, Q2 MJD31C, Q3 IPD50R3K0CE, Q4 MJD31C, Q5 MMBTA42, Q6 MMBTA42, Q7 MMBTA42, Q8 MMBTA42, T1 FL2015-3LB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

Commit message: Library name juggling
Parts:
- T1: value FL2015-3LB -> FL2015; footprint FL2015-3LB:FL2015-4LB -> FL2015:FL2015-4LB
- TT1: value FL2015-3LB -> FL2015; footprint FL2015-3LB:G23736 -> FL2015:G23736
Changed lines of the file:
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@@
   (general
     (thickness 1.6)
-    (drawings 58)
+    (drawings 57)
     (tracks 552)
     (zones 0)
@@
   )
   (setup
-    (last_trace_width 0.508)
+    (last_trace_width 0.25)
     (user_trace_width 0.254)
     (user_trace_width 0.3048)
@@
     (add_net "Net-(U4-Pad8)")
   )
-  (module FL2015-3LB:FL2015-4LB (layer F.Cu)
+  (module FL2015:G23736 (layer F.Cu)
+    (at 139 98 270)
+    (fp_text reference TT1 (at 11.75 8.75 270) (layer F.SilkS)
+      (effects (font (size 1 1) (thickness 0.15)))
+    )
+    (fp_text value FL2015 (at -3.556 8.636 270) (layer Edge.Cuts)
+      (effects (font (size 1 1) (thickness 0.15)))
+    )
+    (fp_line (start 8 6) (end 8 -6) (layer Edge.Cuts) (width 0.12))
+    (fp_line (start -8 6) (end 8 6) (layer Edge.Cuts) (width 0.12))
+    (fp_line (start -8 -6) (end -8 6) (layer Edge.Cuts) (width 0.12))
+    (fp_line (start 8 -6) (end -8 -6) (layer Edge.Cuts) (width 0.12))
+    (fp_line (start -12.75 7.75) (end 12.75 7.75) (layer B.SilkS) (width 0.12))
+    (fp_line (start 12.75 -7.75) (end -12.75 -7.75) (layer B.SilkS) (width 0.12))
+    (fp_line (start -12.75 7.75) (end -12.75 -7.75) (layer B.SilkS) (width 0.12))
+    (fp_line (start 12.75 -7.75) (end 12.75 7.75) (layer B.SilkS) (width 0.12))
+    (pad 9 smd roundrect (at -10.635 5.08 270) (size 5 1.27) (layers B.Cu B.Paste B.Mask) (roundrect_rratio 0.25)
+      (net 26 "Net-(D6-Pad1)"))
+    (pad 8 smd roundrect (at -10.635 -5.08 270) (size 5 1.27) (layers B.Cu B.Paste B.Mask) (roundrect_rratio 0.25)
+      (net 25 "Net-(D4-Pad1)"))
+    (pad 4 smd roundrect (at 10.635 5.08 270) (size 5 1.27) (layers B.Cu B.Paste B.Mask) (roundrect_rratio 0.25)
+      (net 45 "Net-(Q2-Pad1)"))
+    (pad 3 smd roundrect (at 10.635 0 270) (size 5 1.27) (layers B.Cu B.Paste B.Mask) (roundrect_rratio 0.25)
+      (net 13 "Net-(C11-Pad1)"))
+    (pad 5 smd roundrect (at 10.635 -2.54 270) (size 5 1.27) (layers B.Cu B.Paste B.Mask) (roundrect_rratio 0.25)
+      (net 17 "Net-(C20-Pad2)"))
+    (pad 2 smd roundrect (at 10.635 -5.08 270) (size 5 1.27) (layers B.Cu B.Paste B.Mask) (roundrect_rratio 0.25)
+      (net 47 "Net-(Q4-Pad1)"))
+    (pad 1 smd roundrect (at 10.635 2.54 270) (size 5 1.27) (layers B.Cu B.Paste B.Mask) (roundrect_rratio 0.25)
+      (net 18 "Net-(C20-Pad1)"))
+  )
+  (module FL2015:FL2015-4LB (layer F.Cu)
     (at 139 98 270)
     (fp_text reference T1 (at 11.75 8.75 270) (layer F.SilkS)
       (effects (font (size 1 1) (thickness 0.15)))
     )
-    (fp_text value FL2015-3LB (at 0 -0.5 270) (layer F.Fab)
+    (fp_text value FL2015 (at 0 -0.5 270) (layer F.Fab)
       (effects (font (size 1 1) (thickness 0.15)))
     )
@@
     )
   )
-  (module FL2015-3LB:G23736 (layer F.Cu)
-    (at 139 98 270)
-    (fp_text reference TT1 (at 11.75 8.75 270) (layer F.SilkS) hide
-      (effects (font (size 1 1) (thickness 0.15)))
-    )
-    (fp_text value FL2015-3LB (at -3.556 8.636 270) (layer F.Fab)
-      (effects (font (size 1 1) (thickness 0.15)))
-    )
-    (fp_line (start 8 6) (end 8 -6) (layer Edge.Cuts) (width 0.12))
-    (fp_line (start -8 6) (end 8 6) (layer Edge.Cuts) (width 0.12))
-    (fp_line (start -8 -6) (end -8 6) (layer Edge.Cuts) (width 0.12))
-    (fp_line (start 8 -6) (end -8 -6) (layer Edge.Cuts) (width 0.12))
-    (fp_line (start -12.75 7.75) (end 12.75 7.75) (layer B.SilkS) (width 0.12))
-    (fp_line (start 12.75 -7.75) (end -12.75 -7.75) (layer B.SilkS) (width 0.12))
-    (fp_line (start -12.75 7.75) (end -12.75 -7.75) (layer B.SilkS) (width 0.12))
-    (fp_line (start 12.75 -7.75) (end 12.75 7.75) (layer B.SilkS) (width 0.12))
-    (pad 9 smd roundrect (at -10.635 5.08 270) (size 5 1.27) (layers B.Cu B.Paste B.Mask) (roundrect_rratio 0.25)
-      (net 26 "Net-(D6-Pad1)"))
-    (pad 8 smd roundrect (at -10.635 -5.08 270) (size 5 1.27) (layers B.Cu B.Paste B.Mask) (roundrect_rratio 0.25)
-      (net 25 "Net-(D4-Pad1)"))
-    (pad 4 smd roundrect (at 10.635 5.08 270) (size 5 1.27) (layers B.Cu B.Paste B.Mask) (roundrect_rratio 0.25)
-      (net 45 "Net-(Q2-Pad1)"))
-    (pad 3 smd roundrect (at 10.635 0 270) (size 5 1.27) (layers B.Cu B.Paste B.Mask) (roundrect_rratio 0.25)
-      (net 13 "Net-(C11-Pad1)"))
-    (pad 5 smd roundrect (at 10.635 -2.54 270) (size 5 1.27) (layers B.Cu B.Paste B.Mask) (roundrect_rratio 0.25)
-      (net 17 "Net-(C20-Pad2)"))
-    (pad 2 smd roundrect (at 10.635 -5.08 270) (size 5 1.27) (layers B.Cu B.Paste B.Mask) (roundrect_rratio 0.25)
-      (net 47 "Net-(Q4-Pad1)"))
-    (pad 1 smd roundrect (at 10.635 2.54 270) (size 5 1.27) (layers B.Cu B.Paste B.Mask) (roundrect_rratio 0.25)
-      (net 18 "Net-(C20-Pad1)"))
-  )
   (module Resistor_SMD:R_0603_1608Metric (layer F.Cu)
     (at 100 83 90)
@@
     )
   )
-  (gr_arc (start 100 100) (end 64 73.000001) (angle -119) (layer F.SilkS) (width 0.381))
   (gr_text "Sig Out" (at 61.976 88.392 -90) (layer F.SilkS)
     (effects (font (size 1 1) (thickness 0.15)))
@@
   (segment (start 109.75134 131.25) (end 109.25 131.25) (width 0.381) (layer F.Cu) (net 11))
   (segment (start 113.03 129.032) (end 111.96934 129.032) (width 0.381) (layer F.Cu) (net 11))
-  (via (at 138.1 113.25) (size 0.8) (drill 0.4) (layers F.Cu B.Cu) (net 13))
-  (segment (start 139 112.35) (end 138.1 113.25) (width 1.27) (layer B.Cu) (net 13))
-  (segment (start 139 108.635) (end 139 112.35) (width 1.27) (layer B.Cu) (net 13))
-  (segment (start 137.75 112.9) (end 138.1 113.25) (width 1.27) (layer F.Cu) (net 13))
-  (segment (start 137.75 109.4325) (end 137.75 112.9) (width 1.27) (layer F.Cu) (net 13))
   (segment (start 111.184183 73.203476) (end 119.434183 63.553476) (width 0.508) (layer B.Cu) (net 12))
   (segment (start 62.118183 72.3125) (end 62.037728 72.232045) (width 0.508) (layer F.Cu) (net 12))
@@
   (segment (start 93.9225 72.3125) (end 94 72.39) (width 0.381) (layer F.Cu) (net 12))
   (segment (start 90.25 72.3125) (end 93.9225 72.3125) (width 0.381) (layer F.Cu) (net 12))
+  (via (at 138.1 113.25) (size 0.8) (drill 0.4) (layers F.Cu B.Cu) (net 13))
+  (segment (start 139 112.35) (end 138.1 113.25) (width 1.27) (layer B.Cu) (net 13))
+  (segment (start 139 108.635) (end 139 112.35) (width 1.27) (layer B.Cu) (net 13))
+  (segment (start 137.75 112.9) (end 138.1 113.25) (width 1.27) (layer F.Cu) (net 13))
+  (segment (start 137.75 109.4325) (end 137.75 112.9) (width 1.27) (layer F.Cu) (net 13))
   (segment (start 117.4375 126.5) (end 119.5625 126.5) (width 1.27) (layer F.Cu) (net 13))
   (segment (start 119.5625 126.5) (end 119.5625 121.6875) (width 1.27) (layer F.Cu) (net 13))
