File: base/base.sch (KiCad schematic (older format))
At the start: 108 parts, among them J1 Screw_Terminal_01x02, J2 Out, Q1 MSB92W, Q2 MJD31C, Q3 IPD50R3K0CE, Q4 MJD31C, Q5 MMBTA42, Q6 MMBTA42, Q7 MMBTA42, Q8 MMBTA42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

Commit message: Backup
Parts:
- D2: footprint Diode_THT:D_DO-41_SOD81_P10.16mm_Horizontal -> Diode_SMD:D_SMB
Changed lines of the file:
@@
 F 0 "D2" H 1650 6934 50  0000 C CNN
 F 1 "1N4007" H 1650 7025 50  0000 C CNN
-F 2 "Diode_THT:D_DO-41_SOD81_P10.16mm_Horizontal" H 1650 6975 50  0001 C CNN
+F 2 "Diode_SMD:D_SMB" H 1650 6975 50  0001 C CNN
 F 3 "http://www.vishay.com/docs/88503/1n4001.pdf" H 1650 7150 50  0001 C CNN
 	1    1650 7150

Commit message: Added optional G23736 (electronic goldmine) footprint
Parts:
- added TT1: FL2015-3LB, FL2015-3LB:G23736, symbol Device:FL2015-3LB
- C10: value 15n -> 10n; footprint Capacitor_THT:C_Rect_L31.5mm_W11.0mm_P27.50mm_MKS4 -> Capacitor_THT:C_Disc_D10.5mm_W5.0mm_P7.50mm
- C17: value 33n -> 10n; footprint Capacitor_THT:C_Rect_L31.5mm_W11.0mm_P27.50mm_MKS4 -> Capacitor_THT:C_Disc_D10.5mm_W5.0mm_P7.50mm
- R20: value 10k -> 0
Connections:
- wire segments 227 -> 231
Other:
- moved on the sheet: R20
Changed lines of the file:
@@
 Wire Wire Line
 	5550 3300 5700 3300
-Wire Wire Line
-	6050 3500 6050 3000
 $Comp
 L Device:R R23
@@
 Wire Wire Line
 	4750 3100 4750 3500
-Wire Wire Line
-	4750 3100 5850 3100
-Wire Wire Line
-	5850 3000 5850 3100
 $Comp
 L Device:L L1
@@
 $EndComp
 $Comp
-L Device:C C17
-U 1 1 5CB7F2DD
-P 5000 1400
-F 0 "C17" H 4850 1500 50  0000 L CNN
-F 1 "33n" H 4800 1300 50  0000 L CNN
-F 2 "Capacitor_THT:C_Rect_L31.5mm_W11.0mm_P27.50mm_MKS4" H 5038 1250 50  0001 C CNN
-F 3 "~" H 5000 1400 50  0001 C CNN
-	1    5000 1400
-	1    0    0    -1
-$EndComp
-$Comp
-L Device:C C10
-U 1 1 5CB7FB95
-P 3650 1400
-F 0 "C10" H 3500 1500 50  0000 L CNN
-F 1 "15n" H 3500 1300 50  0000 L CNN
-F 2 "Capacitor_THT:C_Rect_L31.5mm_W11.0mm_P27.50mm_MKS4" H 3688 1250 50  0001 C CNN
-F 3 "~" H 3650 1400 50  0001 C CNN
-	1    3650 1400
-	1    0    0    -1
-$EndComp
-$Comp
 L Device:R R24
 U 1 1 5CB7FFB0
@@
 	5550 1650 5550 1250
 Connection ~ 5550 1650
-Wire Wire Line
-	5000 1250 4900 1250
-Wire Wire Line
-	3750 1250 3650 1250
 $Comp
 L power:GND #PWR0105
@@
 L power:GND #PWR0106
 U 1 1 5CB94FE4
-P 3650 1550
-F 0 "#PWR0106" H 3650 1300 50  0001 C CNN
-F 1 "GND" H 3655 1377 50  0000 C CNN
-F 2 "" H 3650 1550 50  0001 C CNN
-F 3 "" H 3650 1550 50  0001 C CNN
-	1    3650 1550
+P 3850 1550
+F 0 "#PWR0106" H 3850 1300 50  0001 C CNN
+F 1 "GND" H 3855 1377 50  0000 C CNN
+F 2 "" H 3850 1550 50  0001 C CNN
+F 3 "" H 3850 1550 50  0001 C CNN
+	1    3850 1550
 	-1   0    0    -1
 $EndComp
 Text GLabel 2100 1250 0    50   Output ~ 0
 -HV
-Connection ~ 3650 1250
 Wire Wire Line
 	5550 2050 5550 2200
@@
 U 1 1 5CF5425C
 P 6700 1400
-F 0 "R30" H 6550 1450 50  0000 L CNN
+F 0 "R30" H 6500 1450 50  0000 L CNN
 F 1 "1M" H 6550 1350 50  0000 L CNN
 F 2 "Resistor_SMD:R_0805_2012Metric" V 6630 1400 50  0001 C CNN
@@
 U 1 1 5CF55E85
 P 6700 1800
-F 0 "R31" H 6550 1850 50  0000 L CNN
+F 0 "R31" H 6500 1850 50  0000 L CNN
 F 1 "1M" H 6550 1750 50  0000 L CNN
 F 2 "Resistor_SMD:R_0805_2012Metric" V 6630 1800 50  0001 C CNN
@@
 U 1 1 5CF5664D
 P 6700 2200
-F 0 "R32" H 6550 2250 50  0000 L CNN
+F 0 "R32" H 6500 2250 50  0000 L CNN
 F 1 "1M" H 6550 2150 50  0000 L CNN
 F 2 "Resistor_SMD:R_0805_2012Metric" V 6630 2200 50  0001 C CNN
@@
 U 1 1 5CF56DCE
 P 6700 2600
-F 0 "R33" H 6550 2650 50  0000 L CNN
+F 0 "R33" H 6500 2650 50  0000 L CNN
 F 1 "1M" H 6550 2550 50  0000 L CNN
 F 2 "Resistor_SMD:R_0805_2012Metric" V 6630 2600 50  0001 C CNN
@@
 U 1 1 5CFC97AB
 P 6700 3150
-F 0 "R34" H 6550 3200 50  0000 L CNN
+F 0 "R34" H 6500 3200 50  0000 L CNN
 F 1 "1M" H 6550 3100 50  0000 L CNN
 F 2 "Resistor_SMD:R_0805_2012Metric" V 6630 3150 50  0001 C CNN
@@
 L Device:R R20
 U 1 1 5D263EF4
-P 3900 1250
-F 0 "R20" V 3800 1250 50  0000 L CNN
-F 1 "10k" V 3900 1200 50  0000 L CNN
-F 2 "Resistor_SMD:R_0805_2012Metric" V 3830 1250 50  0001 C CNN
-F 3 "~" H 3900 1250 50  0001 C CNN
-	1    3900 1250
+P 4350 650
+F 0 "R20" V 4250 650 50  0000 L CNN
+F 1 "0" V 4350 650 50  0000 L CNN
+F 2 "Resistor_SMD:R_0805_2012Metric" V 4280 650 50  0001 C CNN
+F 3 "~" H 4350 650 50  0001 C CNN
+	1    4350 650
 	0    1    1    0
 $EndComp
@@
 Wire Wire Line
 	4100 1350 4100 1250
-Wire Wire Line
-	4050 1250 4100 1250
 Connection ~ 4100 1250
-$Comp
-L Diode:BZX84Cxx D3
-U 1 1 5D303FBE
-P 4350 850
-F 0 "D3" H 4350 1066 50  0000 C CNN
-F 1 "BZX84C47" H 4350 975 50  0000 C CNN
-F 2 "Diode_SMD:D_SOT-23_ANK" H 4350 675 50  0001 C CNN
-F 3 "https://diotec.com/tl_files/diotec/files/pdf/datasheets/bzx84c2v4.pdf" H 4350 850 50  0001 C CNN
-	1    4350 850
-	1    0    0    -1
-$EndComp
-Wire Wire Line
-	5000 1250 5550 1250
-Connection ~ 5000 1250
 Wire Wire Line
 	4600 1250 4550 1250
-Wire Wire Line
-	4500 850  4600 850
-Wire Wire Line
-	4600 850  4600 1250
 Connection ~ 4600 1250
-Wire Wire Line
-	4200 850  4100 850
-Wire Wire Line
-	4100 850  4100 1250
 Text Notes 2450 5700 0    50   ~ 0
 5v5
@@
 $EndComp
 Wire Wire Line
-	6000 3500 6050 3500
-Wire Wire Line
 	5100 3700 5400 3700
 Wire Wire Line
@@
 	2650 3200 2650 3350
 Wire Wire Line
-	2350 1250 3650 1250
-Wire Wire Line
 	2350 1250 2350 2000
 Wire Wire Line
@@
 Wire Wire Line
 	4550 6300 4750 6300
+Wire Wire Line
+	4200 650  4100 650
+Wire Wire Line
+	4500 650  4600 650
+Wire Wire Line
+	4200 950  4100 950
+Wire Wire Line
+	4100 950  4100 1250
+Wire Wire Line
+	4500 950  4600 950
+Wire Wire Line
+	4600 950  4600 1250
+Connection ~ 4100 950
+Connection ~ 4600 950
+$Comp
+L Diode:BZX84Cxx D3
+U 1 1 5D303FBE
+P 4350 950
+F 0 "D3" H 4350 1166 50  0000 C CNN
+F 1 "BZX84C47" H 4350 1075 50  0000 C CNN
+F 2 "Diode_SMD:D_SOT-23_ANK" H 4350 775 50  0001 C CNN
+F 3 "https://diotec.com/tl_files/diotec/files/pdf/datasheets/bzx84c2v4.pdf" H 4350 950 50  0001 C CNN
+	1    4350 950
+	1    0    0    -1
+$EndComp
+Wire Wire Line
+	4100 650  4100 950
+Wire Wire Line
+	4600 650  4600 950
+$Comp
+L Device:C C10
+U 1 1 5CE22DE7
+P 3850 1400
+F 0 "C10" H 3700 1500 50  0000 L CNN
+F 1 "10n" H 3700 1300 50  0000 L CNN
+F 2 "Capacitor_THT:C_Disc_D10.5mm_W5.0mm_P7.50mm" H 3888 1250 50  0001 C CNN
+F 3 "~" H 3850 1400 50  0001 C CNN
+	1    3850 1400
+	1    0    0    -1
+$EndComp
+$Comp
+L Device:C C17
+U 1 1 5CE233CF
+P 5000 1400
+F 0 "C17" H 4850 1500 50  0000 L CNN
+F 1 "10n" H 4850 1300 50  0000 L CNN
+F 2 "Capacitor_THT:C_Disc_D10.5mm_W5.0mm_P7.50mm" H 5038 1250 50  0001 C CNN
+F 3 "~" H 5000 1400 50  0001 C CNN
+	1    5000 1400
+	1    0    0    -1
+$EndComp
+Wire Wire Line
+	4900 1250 5000 1250
+Connection ~ 5000 1250
+Wire Wire Line
+	5000 1250 5550 1250
+Connection ~ 3850 1250
+Wire Wire Line
+	3850 1250 4100 1250
+Wire Wire Line
+	6050 3100 6050 3000
+Wire Wire Line
+	4750 3100 6050 3100
+Wire Wire Line
+	2350 1250 3850 1250
+Wire Wire Line
+	5850 3000 5850 3250
+Wire Wire Line
+	5850 3250 6000 3250
+Wire Wire Line
+	6000 3250 6000 3500
+$Comp
+L Device:FL2015-3LB TT1
+U 1 1 5CEA8266
+P 5600 2600
+F 0 "TT1" V 5800 2300 50  0000 R CNN
+F 1 "FL2015-3LB" V 5550 3600 50  0000 R CNN
+F 2 "FL2015-3LB:G23736" H 7250 1150 50  0001 C CNN
+F 3 "" H 7250 1150 50  0001 C CNN
+	1    5600 2600
+	0    -1   -1   0
+$EndComp
+Connection ~ 5100 3000
+Connection ~ 5850 3000
+Connection ~ 5400 3000
+Connection ~ 6050 3000
+Connection ~ 5700 3000
+Connection ~ 5250 2200
+Connection ~ 5850 2200
 $EndSCHEMATC

Commit message: More routing. Removed excessive ripper remover
Parts:
- removed C10, C15: 10n, Capacitor_THT:C_Disc_D10.5mm_W5.0mm_P7.50mm, symbol Device:C
- removed D3: BZX84C47, Diode_SMD:D_SOT-23_ANK, symbol Diode:BZX84Cxx
- removed Q1: MSB92W, Package_TO_SOT_SMD:SOT-23, symbol Transistor_BJT:MMBT3906
- removed R20: 0, Resistor_SMD:R_0805_2012Metric, symbol Device:R
- removed R21: 10M, Resistor_SMD:R_0805_2012Metric, symbol Device:R
- removed R24: 10k, Resistor_SMD:R_0805_2012Metric, symbol Device:R
- RV1: footprint (none) -> Potentiometer_SMD:Potentiometer_Bourns_3314J_Vertical
- U1: footprint (none) -> Package_TO_SOT_SMD:SOT-223-3_TabPin2
- U2: footprint (none) -> Package_SO:SOIC-8_3.9x4.9mm_P1.27mm
Connections:
- wire segments 231 -> 215
Changed lines of the file:
@@
 	1    0    0    -1
-$EndComp
-$Comp
-L Device:R R24
-U 1 1 5CB7FFB0
-P 4750 1250
-F 0 "R24" V 4650 1250 50  0000 L CNN
-F 1 "10k" V 4750 1200 50  0000 L CNN
-F 2 "Resistor_SMD:R_0805_2012Metric" V 4680 1250 50  0001 C CNN
-F 3 "~" H 4750 1250 50  0001 C CNN
-	1    4750 1250
-	0    1    1    0
 $EndComp
 Wire Wire Line
@@
 	-1   0    0    -1
 $EndComp
-$Comp
-L power:GND #PWR0106
-U 1 1 5CB94FE4
-P 3850 1550
-F 0 "#PWR0106" H 3850 1300 50  0001 C CNN
-F 1 "GND" H 3855 1377 50  0000 C CNN
-F 2 "" H 3850 1550 50  0001 C CNN
-F 3 "" H 3850 1550 50  0001 C CNN
-	1    3850 1550
-	-1   0    0    -1
-$EndComp
 Text GLabel 2100 1250 0    50   Output ~ 0
 -HV
@@
 F 0 "U2" H 4100 4350 50  0000 C CNN
 F 1 "LM358" H 4050 4350 50  0001 C CNN
-F 2 "" H 3950 4200 50  0001 C CNN
+F 2 "Package_SO:SOIC-8_3.9x4.9mm_P1.27mm" H 3950 4200 50  0001 C CNN
 F 3 "http://www.ti.com/lit/ds/symlink/lm2904-n.pdf" H 3950 4200 50  0001 C CNN
 	1    3950 4200
@@
 F 0 "U2" H 2650 3900 50  0000 C CNN
 F 1 "LM358" H 2600 4100 50  0000 C CNN
-F 2 "" H 2650 4100 50  0001 C CNN
+F 2 "Package_SO:SOIC-8_3.9x4.9mm_P1.27mm" H 2650 4100 50  0001 C CNN
 F 3 "http://www.ti.com/lit/ds/symlink/lm2904-n.pdf" H 2650 4100 50  0001 C CNN
 	2    2650 4100
@@
 F 0 "U2" H 3650 3950 50  0001 L CNN
 F 1 "LM358" H 3800 4200 50  0000 L CNN
-F 2 "" H 3950 4200 50  0001 C CNN
+F 2 "Package_SO:SOIC-8_3.9x4.9mm_P1.27mm" H 3950 4200 50  0001 C CNN
 F 3 "http://www.ti.com/lit/ds/symlink/lm2904-n.pdf" H 3950 4200 50  0001 C CNN
 	3    3950 4200
@@
 F 0 "U1" H 1300 5942 50  0000 C CNN
 F 1 "LM1117-ADJ" H 1300 5851 50  0000 C CNN
-F 2 "" H 1300 5700 50  0001 C CNN
+F 2 "Package_TO_SOT_SMD:SOT-223-3_TabPin2" H 1300 5700 50  0001 C CNN
 F 3 "http://www.ti.com/lit/ds/symlink/lm1117.pdf" H 1300 5700 50  0001 C CNN
 	1    1300 5700
@@
 F 0 "RV1" H 1130 3646 50  0000 R CNN
 F 1 "10k" H 1130 3555 50  0000 R CNN
-F 2 "" H 1200 3600 50  0001 C CNN
+F 2 "Potentiometer_SMD:Potentiometer_Bourns_3314J_Vertical" H 1200 3600 50  0001 C CNN
 F 3 "~" H 1200 3600 50  0001 C CNN
 	1    1200 3600
@@
 Wire Wire Line
 	7750 2450 8000 2450
-$Comp
-L Transistor_BJT:MMBT3906 Q1
-U 1 1 5D1EBA2E
-P 4350 1350
-F 0 "Q1" V 4678 1350 50  0000 C CNN
-F 1 "MSB92W" V 4587 1350 50  0000 C CNN
-F 2 "Package_TO_SOT_SMD:SOT-23" H 4550 1275 50  0001 L CIN
-F 3 "https://www.fairchildsemi.com/datasheets/2N/2N3906.pdf" H 4350 1350 50  0001 L CNN
-	1    4350 1350
-	0    1    -1   0
-$EndComp
 Wire Wire Line
 	4450 2500 4450 3050
@@
 	4050 2500 4450 2500
 Connection ~ 4450 3050
-$Comp
-L Device:R R20
-U 1 1 5D263EF4
-P 4350 650
-F 0 "R20" V 4250 650 50  0000 L CNN
-F 1 "0" V 4350 650 50  0000 L CNN
-F 2 "Resistor_SMD:R_0805_2012Metric" V 4280 650 50  0001 C CNN
-F 3 "~" H 4350 650 50  0001 C CNN
-	1    4350 650
-	0    1    1    0
-$EndComp
-Wire Wire Line
-	4100 1250 4150 1250
-$Comp
-L Device:R R21
-U 1 1 5D28922D
-P 4100 1500
-F 0 "R21" H 4170 1546 50  0000 L CNN
-F 1 "10M" H 4170 1455 50  0000 L CNN
-F 2 "Resistor_SMD:R_0805_2012Metric" V 4030 1500 50  0001 C CNN
-F 3 "~" H 4100 1500 50  0001 C CNN
-	1    4100 1500
-	1    0    0    -1
-$EndComp
-$Comp
-L Device:C C15
-U 1 1 5D289BAC
-P 4350 1850
-F 0 "C15" H 4200 1950 50  0000 L CNN
-F 1 "10n" H 4200 1750 50  0000 L CNN
-F 2 "Capacitor_THT:C_Disc_D10.5mm_W5.0mm_P7.50mm" H 4388 1700 50  0001 C CNN
-F 3 "~" H 4350 1850 50  0001 C CNN
-	1    4350 1850
-	1    0    0    -1
-$EndComp
-$Comp
-L power:GND #PWR02
-U 1 1 5D28A1CD
-P 4350 2000
-F 0 "#PWR02" H 4350 1750 50  0001 C CNN
-F 1 "GND" H 4355 1827 50  0000 C CNN
-F 2 "" H 4350 2000 50  0001 C CNN
-F 3 "" H 4350 2000 50  0001 C CNN
-	1    4350 2000
-	-1   0    0    -1
-$EndComp
-Wire Wire Line
-	4350 1700 4350 1650
-Wire Wire Line
-	4100 1650 4350 1650
-Connection ~ 4350 1650
-Wire Wire Line
-	4350 1650 4350 1550
-Wire Wire Line
-	4100 1350 4100 1250
-Connection ~ 4100 1250
-Wire Wire Line
-	4600 1250 4550 1250
-Connection ~ 4600 1250
 Text Notes 2450 5700 0    50   ~ 0
 5v5
@@
 Wire Wire Line
 	2350 1250 2100 1250
-Connection ~ 2350 1250
 $Comp
 L power:GND #PWR0111
@@
 Wire Wire Line
 	4550 6300 4750 6300
-Wire Wire Line
-	4200 650  4100 650
-Wire Wire Line
-	4500 650  4600 650
-Wire Wire Line
-	4200 950  4100 950
-Wire Wire Line
-	4100 950  4100 1250
-Wire Wire Line
-	4500 950  4600 950
-Wire Wire Line
-	4600 950  4600 1250
-Connection ~ 4100 950
-Connection ~ 4600 950
-$Comp
-L Diode:BZX84Cxx D3
-U 1 1 5D303FBE
-P 4350 950
-F 0 "D3" H 4350 1166 50  0000 C CNN
-F 1 "BZX84C47" H 4350 1075 50  0000 C CNN
-F 2 "Diode_SMD:D_SOT-23_ANK" H 4350 775 50  0001 C CNN
-F 3 "https://diotec.com/tl_files/diotec/files/pdf/datasheets/bzx84c2v4.pdf" H 4350 950 50  0001 C CNN
-	1    4350 950
-	1    0    0    -1
-$EndComp
-Wire Wire Line
-	4100 650  4100 950
-Wire Wire Line
-	4600 650  4600 950
-$Comp
-L Device:C C10
-U 1 1 5CE22DE7
-P 3850 1400
-F 0 "C10" H 3700 1500 50  0000 L CNN
-F 1 "10n" H 3700 1300 50  0000 L CNN
-F 2 "Capacitor_THT:C_Disc_D10.5mm_W5.0mm_P7.50mm" H 3888 1250 50  0001 C CNN
-F 3 "~" H 3850 1400 50  0001 C CNN
-	1    3850 1400
-	1    0    0    -1
-$EndComp
 $Comp
 L Device:C C17
@@
 	1    0    0    -1
 $EndComp
-Wire Wire Line
-	4900 1250 5000 1250
 Connection ~ 5000 1250
 Wire Wire Line
 	5000 1250 5550 1250
-Connection ~ 3850 1250
-Wire Wire Line
-	3850 1250 4100 1250
 Wire Wire Line
 	6050 3100 6050 3000
 Wire Wire Line
 	4750 3100 6050 3100
-Wire Wire Line
-	2350 1250 3850 1250
 Wire Wire Line
 	5850 3000 5850 3250
@@
 Connection ~ 5250 2200
 Connection ~ 5850 2200
+Wire Wire Line
+	2350 1250 5000 1250
+Connection ~ 2350 1250
 $EndSCHEMATC

Commit message: Accidentally used PNP bjt's for royer drivers
Parts:
- Q2, Q4: symbol Transistor_BJT:BCP53 -> Transistor_BJT:BD249
Connections:
- net at C20.1, Q2.2 (C), T1.1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: no longer Q2.4 (C)
- net at C20.2, Q4.2 (C), T1.5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: no longer Q4.4 (C)
Changed lines of the file:
@@
 $EndComp
 $Comp
-L Transistor_BJT:BCP53 Q2
+L Transistor_BJT:BD249 Q2
 U 1 1 5CC76357
 P 5000 3500
@@
 Connection ~ 5700 3300
 $Comp
-L Transistor_BJT:BCP53 Q4
+L Transistor_BJT:BD249 Q4
 U 1 1 5CC7DF8F
 P 5800 3500

Commit message: Moved stuff around. Added isolation slots.
Parts:
- J2: footprint Connector_Coaxial:SMA_Amphenol_901-144_Vertical -> Connector_Coaxial:SMA_Amphenol_132291-12_Vertical
Changed lines of the file:
@@
 F 0 "J2" H 10950 1975 50  0000 L CNN
 F 1 "Out" H 10950 1884 50  0000 L CNN
-F 2 "Connector_Coaxial:SMA_Amphenol_901-144_Vertical" H 10850 2000 50  0001 C CNN
+F 2 "Connector_Coaxial:SMA_Amphenol_132291-12_Vertical" H 10850 2000 50  0001 C CNN
 F 3 " ~" H 10850 2000 50  0001 C CNN
 	1    10850 2000
