File: base/base.sch (KiCad schematic (older format))
At the start: 108 parts, among them J1 Screw_Terminal_01x02, J2 Out, Q2 MJD31C, Q3 IPD50R3K0CE, Q4 MJD31C, Q5 MMBTA42, Q6 MMBTA42, Q7 MMBTA42, Q8 MMBTA42, T1 FL2015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

Commit message: Fixed undriven pins errors in DRC
Other:
- moved on the sheet: C21, C22, C23, C24, D10, D11, D8, D9, Q5, Q6, Q7, Q8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
