File: base.kicad_pcb (KiCad board)
At the start: 2 copper layers, 100 x 100 mm, 109 parts, among them J1 Screw_Terminal_01x02, J2 Out, Q2 MJD31C, Q3 IPD50R3K0CE, Q4 MJD31C, Q5 MMBTA42, Q6 MMBTA42, Q7 MMBTA42, Q8 MMBTA42, T1 FL2015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

Commit message: moved files around. Changed cutout for alternative transformer package
Parts:
- added HV1: Symbol_Highvoltage_Type2_SilkScreenTop_Small, HvSymbol:Symbol_Highvoltage_Type2_SilkScreenTop_Small, F.Cu at (108.5, 67.1)
Routing:
- net Net-(C11-Pad1): track 43.3 -> 44.5 mm
- net Net-(L1-Pad2): vias 0 -> 1
- net Net-(L1-Pad1): vias 0 -> 1
Changed lines of the file:
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@@
   (general
     (thickness 1.6)
-    (drawings 57)
-    (tracks 552)
+    (drawings 58)
+    (tracks 556)
     (zones 0)
-    (modules 109)
+    (modules 110)
     (nets 69)
   )
@@
   )
   (setup
-    (last_trace_width 0.25)
+    (last_trace_width 0.635)
     (user_trace_width 0.254)
     (user_trace_width 0.3048)
@@
       (effects (font (size 1 1) (thickness 0.15)))
     )
-    (fp_line (start 8 6) (end 8 -6) (layer Edge.Cuts) (width 0.12))
-    (fp_line (start -8 6) (end 8 6) (layer Edge.Cuts) (width 0.12))
-    (fp_line (start -8 -6) (end -8 6) (layer Edge.Cuts) (width 0.12))
-    (fp_line (start 8 -6) (end -8 -6) (layer Edge.Cuts) (width 0.12))
+    (fp_line (start 8 8) (end 8 -8) (layer Edge.Cuts) (width 0.12))
+    (fp_line (start -8 8) (end 8 8) (layer Edge.Cuts) (width 0.12))
+    (fp_line (start -8 -8) (end -8 8) (layer Edge.Cuts) (width 0.12))
+    (fp_line (start 8 -8) (end -8 -8) (layer Edge.Cuts) (width 0.12))
     (fp_line (start -12.75 7.75) (end 12.75 7.75) (layer B.SilkS) (width 0.12))
     (fp_line (start 12.75 -7.75) (end -12.75 -7.75) (layer B.SilkS) (width 0.12))
@@
       (net 18 "Net-(C20-Pad1)"))
   )
+  (module HvSymbol:Symbol_Highvoltage_Type2_SilkScreenTop_Small (layer F.Cu)
+    (at 108.55 67.1)
+    (descr "Symbol, Highvoltage, Type 2, Copper Top, Small,")
+    (tags "Symbol, Highvoltage, Type 2, Copper Top, Small,")
+    (attr virtual)
+    (fp_text reference HV1 (at 0 -10.16) (layer F.Fab) hide
+      (effects (font (size 1 1) (thickness 0.15)))
+    )
+    (fp_text value Symbol_Highvoltage_Type2_SilkScreenTop_Small (at 0 7.62) (layer F.Fab)
+      (effects (font (size 1 1) (thickness 0.15)))
+    )
+    (fp_line (start -1.143 1.397) (end -1.27 0.889) (layer F.SilkS) (width 0.381))
+    (fp_line (start 0 -0.889) (end -1.143 1.397) (layer F.SilkS) (width 0.381))
+    (fp_line (start -1.397 -0.889) (end 0 -0.889) (layer F.SilkS) (width 0.381))
+    (fp_line (start 0.127 -3.175) (end -1.397 -0.889) (layer F.SilkS) (width 0.381))
+    (fp_line (start 0.381 -2.794) (end 0.254 -3.302) (layer F.SilkS) (width 0.381))
+    (fp_line (start 1.143 -3.302) (end 0.381 -2.794) (layer F.SilkS) (width 0.381))
+    (fp_line (start -0.635 -1.27) (end 1.143 -3.302) (layer F.SilkS) (width 0.381))
+    (fp_line (start 0.635 -1.27) (end -0.635 -1.27) (layer F.SilkS) (width 0.381))
+    (fp_line (start -1.143 1.524) (end 0.635 -1.27) (layer F.SilkS) (width 0.381))
+    (fp_line (start -0.635 1.27) (end -1.143 1.524) (layer F.SilkS) (width 0.381))
+    (fp_line (start -1.397 1.905) (end -0.635 1.27) (layer F.SilkS) (width 0.381))
+    (fp_line (start -1.27 0.889) (end -1.397 1.905) (layer F.SilkS) (width 0.381))
+    (fp_line (start -1.016 -1.016) (end 0.254 -1.016) (layer F.SilkS) (width 0.381))
+    (fp_line (start 0.381 -2.921) (end -1.016 -1.016) (layer F.SilkS) (width 0.381))
+    (fp_line (start -8.89 3.81) (end 0 -7.62) (layer F.SilkS) (width 1.27))
+    (fp_line (start 8.89 3.81) (end -8.89 3.81) (layer F.SilkS) (width 1.27))
+    (fp_line (start 0 -7.62) (end 8.89 3.81) (layer F.SilkS) (width 1.27))
+  )
   (module FL2015:FL2015-4LB (layer F.Cu)
     (at 139 98 270)
@@
       (effects (font (size 1 1) (thickness 0.15)))
     )
-    (fp_text value -HV (at 3 0.61) (layer F.SilkS)
+    (fp_text value -HV (at -0.075 2.085) (layer F.SilkS)
       (effects (font (size 1 1) (thickness 0.15)))
     )
@@
     (tags "Diode SMB (DO-214AA)")
     (attr smd)
-    (fp_text reference D2 (at 0 -3 270) (layer F.SilkS)
+    (fp_text reference D2 (at -4.7 0.425) (layer F.SilkS)
       (effects (font (size 1 1) (thickness 0.15)))
     )
@@
     (tags "capacitor tantalum")
     (attr smd)
-    (fp_text reference C3 (at 5.192 2.442) (layer F.SilkS)
+    (fp_text reference C3 (at -5.35 0.05) (layer F.SilkS)
       (effects (font (size 1 1) (thickness 0.15)))
     )
@@
     (tags "Potentiometer vertical Bourns 3314J")
     (attr smd)
-    (fp_text reference RV1 (at 0 -4.25 90) (layer F.SilkS)
+    (fp_text reference RV1 (at 3.1 0 180) (layer F.SilkS)
       (effects (font (size 1 1) (thickness 0.15)))
     )
@@
     (tags "CMS SOT")
     (attr smd)
-    (fp_text reference U1 (at 2.73 4.762 90) (layer F.SilkS)
+    (fp_text reference U1 (at -5.25 -2.05 180) (layer F.SilkS)
       (effects (font (size 1 1) (thickness 0.15)))
     )
@@
     )
   )
+  (gr_circle (center 100 100) (end 127.518176 100) (layer B.Fab) (width 0.12))
   (gr_text "Sig Out" (at 61.976 88.392 -90) (layer F.SilkS)
     (effects (font (size 1 1) (thickness 0.15)))
@@
   (gr_line (start 129.25 68.25) (end 127.5 70.75) (layer Edge.Cuts) (width 0.05))
   (gr_line (start 131.5 69.75) (end 129.25 68.25) (layer Edge.Cuts) (width 0.05))
-  (gr_text "WARNING:\nHIGH VOLTAGE!" (at 99.822 68.58) (layer F.SilkS)
+  (gr_text "WARNING:\nHIGH VOLTAGE!" (at 112.125 56.1) (layer F.SilkS)
     (effects (font (size 1.6256 1.6256) (thickness 0.15)))
   )
@@
     (effects (font (size 1.5 1.5) (thickness 0.3)) (justify mirror))
   )
-  (gr_text "TOP\n" (at 88.75 58.75) (layer F.Cu)
+  (gr_text "TOP\n" (at 87.925 64.4) (layer F.Cu)
     (effects (font (size 1.5 1.5) (thickness 0.3)))
   )
-  (gr_text "PMT B133D01 Base\nTomWimmenhove.com\n1917 Rev A\n\n" (at 112.014 65.024 326.3) (layer F.SilkS)
+  (gr_text "PMT B133D01 Base\nTomWimmenhove.com\n1917 Rev A\n\n" (at 86.875 59.45) (layer F.SilkS)
     (effects (font (size 1 1) (thickness 0.15)))
   )
   (gr_circle (center 100 100) (end 127.518176 100) (layer B.Fab) (width 0.12))
   (gr_circle (center 100 100) (end 101 150) (layer Edge.Cuts) (width 0.05))
+  (via (at 131.5 134.75) (size 2) (drill 1.2) (layers F.Cu B.Cu) (net 33))
   (segment (start 115.0375 143.7875) (end 116.5 143.7875) (width 0.635) (layer F.Cu) (net 1))
   (segment (start 113.405 141.7) (end 113.405 142.155) (width 0.635) (layer F.Cu) (net 1))
@@
   (segment (start 136.75 117.75) (end 137.75 116.75) (width 1.27) (layer B.Cu) (net 13))
   (segment (start 137.75 116.75) (end 137.75 113.6) (width 1.27) (layer B.Cu) (net 13))
+  (segment (start 136.332812 118.786283) (end 136.75 117.75) (width 0.635) (layer F.Cu) (net 13))
   (segment (start 72.492677 121.828464) (end 72.344822 121.976319) (width 0.3048) (layer F.Cu) (net 14))
   (segment (start 72.492677 121.789718) (end 72.492677 121.828464) (width 0.3048) (layer F.Cu) (net 14))
@@
   (via (at 88.15 109.400004) (size 0.8) (drill 0.4) (layers F.Cu B.Cu) (net 20))
   (segment (start 88.15 110.6) (end 88.15 109.400004) (width 0.635) (layer F.Cu) (net 20))
-  (segment (start 96.509297 120.886161) (end 93.675809 120.532376) (width 0.635) (layer F.Cu) (net 20))
   (segment (start 93.675809 118.414191) (end 93.675809 120.532376) (width 0.508) (layer F.Cu) (net 20))
   (segment (start 94.5 116.4) (end 94.5 117.59) (width 0.508) (layer F.Cu) (net 20))
@@
   (segment (start 88.15 114.45) (end 90.1 116.4) (width 0.508) (layer B.Cu) (net 20))
   (segment (start 88.15 109.400004) (end 88.15 114.45) (width 0.508) (layer B.Cu) (net 20))
+  (segment (start 93.675809 120.532376) (end 96.509297 120.886161) (width 0.508) (layer F.Cu) (net 20))
   (segment (start 93.55 113.35) (end 93.55 113.35) (width 0.635) (layer F.Cu) (net 21))
   (segment (start 93.55 114.4) (end 93.55 113.35) (width 0.635) (layer F.Cu) (net 21))
@@
   (segment (start 67.5 92) (end 68.75 93.25) (width 0.381) (layer F.Cu) (net 31))
   (segment (start 133.291385 128.831587) (end 133.479899 129.020101) (width 1.27) (layer F.Cu) (net 32))
-  (segment (start 130.691385 126.231587) (end 133.479899 129.020101) (width 1.27) (layer F.Cu) (net 32))
+  (segment (start 130.691385 126.231587) (end 131.404899 126.945101) (width 1.27) (layer F.Cu) (net 32))
   (segment (start 130.691385 123.770062) (end 130.691385 126.231587) (width 1.27) (layer F.Cu) (net 32))
   (segment (start 133.479899 129.020101) (end 141.791385 123.770062) (width 1.27) (layer F.Cu) (net 32))
+  (segment (start 131.404899 126.945101) (end 133.479899 129.020101) (width 1.27) (layer F.Cu) (net 32))
+  (via (at 131.5 127.25) (size 2) (drill 1.2) (layers F.Cu B.Cu) (net 32))
   (segment (start 128.190202 131.65) (end 129.520101 132.979899) (width 1.27) (layer F.Cu) (net 33))
   (segment (start 121.5 131.65) (end 128.190202 131.65) (width 1.27) (layer F.Cu) (net 33))
@@
   (segment (start 120.393445 110.74476) (end 117.200293 113.716776) (width 0.508) (layer F.Cu) (net 39))
   (segment (start 93.324191 122.067624) (end 90.454558 119.821315) (width 0.508) (layer F.Cu) (net 40))
-  (segment (start 82.799707 115.406459) (end 84.408695 117.015447) (width 0.635) (layer F.Cu) (net 41))
-  (segment (start 82.799707 113.716776) (end 82.799707 115.406459) (width 0.635) (layer F.Cu) (net 41))
+  (segment (start 82.799707 115.406459) (end 82.799707 113.716776) (width 0.508) (layer F.Cu) (net 41))
+  (segment (start 84.408695 117.015447) (end 82.799707 115.406459) (width 0.508) (layer F.Cu) (net 41))
   (segment (start 67.26 104.781) (end 67.26 103.625) (width 0.381) (layer F.Cu) (net 42))
   (segment (start 67.26 107.49) (end 67.26 104.781) (width 0.381) (layer F.Cu) (net 42))

Commit message: Fixed DRC
Parts:
- moved TP1 1.52 mm to (81.1, 124.3)
- moved Q4 0.71 mm to (141.0, 119.5)
- moved Q2 0.65 mm to (129.8, 119.0)
- moved R23 0.55 mm to (124.2, 119.5)
Routing:
- net Net-(C20-Pad1): track 25.3 -> 27.3 mm
- net Net-(Q4-Pad1): track 23.5 -> 24.3 mm
- net Net-(C11-Pad1): track 44.5 -> 43.9 mm
Changed lines of the file:
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@@
     (thickness 1.6)
     (drawings 58)
-    (tracks 556)
+    (tracks 558)
     (zones 0)
     (modules 110)
@@
   )
   (setup
-    (last_trace_width 0.635)
+    (last_trace_width 0.508)
     (user_trace_width 0.254)
     (user_trace_width 0.3048)
@@
     (user_trace_width 1.27)
     (trace_clearance 0.2)
-    (zone_clearance 0.5)
+    (zone_clearance 0.381)
     (zone_45_only no)
     (trace_min 0.2)
@@
   )
   (module TestPoint:TestPoint_Pad_D1.5mm (layer F.Cu)
-    (at 82.042 125.476)
+    (at 81.075 124.3)
     (descr "SMD pad as test Point, diameter 1.5mm")
     (tags "test point SMD pad")
@@
   )
   (module Package_TO_SOT_SMD:TO-252-2 (layer F.Cu)
-    (at 130.4 119 65)
+    (at 129.75 119 65)
     (descr "TO-252 / DPAK SMD package, http://www.infineon.com/cms/en/product/packages/PG-TO252/PG-TO252-3-1/")
     (tags "DPAK TO-252 DPAK-3 TO-252-3 SOT-428")
@@
   )
   (module Package_TO_SOT_SMD:TO-252-2 (layer F.Cu)
-    (at 141.5 119 65)
+    (at 141 119.5 65)
     (descr "TO-252 / DPAK SMD package, http://www.infineon.com/cms/en/product/packages/PG-TO252/PG-TO252-3-1/")
     (tags "DPAK TO-252 DPAK-3 TO-252-3 SOT-428")
@@
   )
   (module Resistor_SMD:R_0805_2012Metric (layer F.Cu)
-    (at 124.75 119.5 245)
+    (at 124.2 119.5 245)
     (descr "Resistor SMD 0805 (2012 Metric), square (rectangular) end terminal, IPC_7351 nominal, (Body size source: https://docs.google.com/spreadsheets/d/1BsfQQcO9C6DZCsRaXUlFlo91Tg2WpOkGARC1WS5S8t0/edit?usp=sharing), generated with kicad-footprint-generator")
     (tags resistor)
@@
   (segment (start 81.1875 130.8125) (end 84.15 127.85) (width 0.381) (layer F.Cu) (net 3))
   (segment (start 84.416 127.85) (end 84.9 127.85) (width 0.381) (layer F.Cu) (net 3))
-  (segment (start 82.042 125.476) (end 84.416 127.85) (width 0.381) (layer F.Cu) (net 3))
+  (segment (start 81.075 124.3) (end 81.075 124.509) (width 0.381) (layer F.Cu) (net 3))
+  (segment (start 81.075 125.0875) (end 79.7 126.4625) (width 0.381) (layer F.Cu) (net 3))
+  (segment (start 81.075 124.3) (end 81.075 125.0875) (width 0.381) (layer F.Cu) (net 3))
   (segment (start 109 142.295) (end 109 143.9625) (width 0.381) (layer F.Cu) (net 4))
   (segment (start 109.595 141.7) (end 109 142.295) (width 0.381) (layer F.Cu) (net 4))
@@
   (segment (start 117.4375 126.5) (end 119.5625 126.5) (width 1.27) (layer F.Cu) (net 13))
   (segment (start 119.5625 126.5) (end 119.5625 121.6875) (width 1.27) (layer F.Cu) (net 13))
-  (segment (start 122.599664 118.650336) (end 125.146205 118.650336) (width 1.27) (layer F.Cu) (net 13))
   (segment (start 119.5625 121.6875) (end 121.875 119.375) (width 1.27) (layer F.Cu) (net 13))
-  (segment (start 121.875 119.375) (end 122.599664 118.650336) (width 1.27) (layer F.Cu) (net 13))
   (via (at 136.75 117.75) (size 0.8) (drill 0.4) (layers F.Cu B.Cu) (net 13))
   (via (at 121.875 119.375) (size 0.8) (drill 0.4) (layers F.Cu B.Cu) (net 13))
@@
   (segment (start 137.75 116.75) (end 137.75 113.6) (width 1.27) (layer B.Cu) (net 13))
   (segment (start 136.332812 118.786283) (end 136.75 117.75) (width 0.635) (layer F.Cu) (net 13))
+  (segment (start 124.150336 118.650336) (end 124.596205 118.650336) (width 1.27) (layer F.Cu) (net 13))
+  (segment (start 121.875 119.375) (end 122.599664 118.650336) (width 1.27) (layer F.Cu) (net 13))
+  (segment (start 122.599664 118.650336) (end 124.150336 118.650336) (width 1.27) (layer F.Cu) (net 13))
   (segment (start 72.492677 121.828464) (end 72.344822 121.976319) (width 0.3048) (layer F.Cu) (net 14))
   (segment (start 72.492677 121.789718) (end 72.492677 121.828464) (width 0.3048) (layer F.Cu) (net 14))
@@
   (segment (start 142.75 110.75) (end 144 112) (width 1.27) (layer F.Cu) (net 17))
   (segment (start 142.75 109.4325) (end 142.75 110.75) (width 1.27) (layer F.Cu) (net 17))
-  (segment (start 144 115.484252) (end 142.387498 117.096754) (width 1.27) (layer F.Cu) (net 17))
-  (segment (start 144 112) (end 144 115.484252) (width 1.27) (layer F.Cu) (net 17))
   (segment (start 141.2875 111.75) (end 142.75 110.75) (width 1.27) (layer F.Cu) (net 17))
   (via (at 142.55 108.1) (size 0.8) (drill 0.4) (layers F.Cu B.Cu) (net 17))
@@
   (segment (start 142.075 108.1) (end 141.54 108.635) (width 1.27) (layer B.Cu) (net 17))
   (segment (start 142.55 108.1) (end 142.075 108.1) (width 1.27) (layer B.Cu) (net 17))
+  (segment (start 141.2875 116.996756) (end 141.887498 117.596754) (width 1.27) (layer F.Cu) (net 17))
+  (segment (start 141.2875 111.75) (end 141.2875 116.996756) (width 1.27) (layer F.Cu) (net 17))
   (segment (start 132.75 108.7) (end 132.75 109.4325) (width 0.381) (layer F.Cu) (net 18))
   (segment (start 133.6 107.85) (end 132.75 108.7) (width 0.381) (layer F.Cu) (net 18))
@@
   (via (at 132.75 113.55) (size 0.8) (drill 0.4) (layers F.Cu B.Cu) (net 18))
   (segment (start 132.75 109.4325) (end 132.75 113.55) (width 1.27) (layer F.Cu) (net 18))
-  (segment (start 132.75 113.55) (end 132.75 115.959256) (width 1.27) (layer F.Cu) (net 18))
   (segment (start 132.8 113.6) (end 132.75 113.55) (width 1.27) (layer B.Cu) (net 18))
   (segment (start 134.7 113.6) (end 132.8 113.6) (width 1.27) (layer B.Cu) (net 18))
@@
   (segment (start 136.46 108.635) (end 136.45 108.645) (width 1.27) (layer B.Cu) (net 18))
   (segment (start 136.45 108.645) (end 136.45 111.85) (width 1.27) (layer B.Cu) (net 18))
+  (segment (start 132.75 114.984252) (end 130.637498 117.096754) (width 1.27) (layer F.Cu) (net 18))
+  (segment (start 132.75 113.55) (end 132.75 114.984252) (width 1.27) (layer F.Cu) (net 18))
   (segment (start 87.615113 117.332675) (end 84.584887 121.267325) (width 0.508) (layer F.Cu) (net 19))
   (segment (start 89.1 112.6) (end 86.6 112.6) (width 0.508) (layer F.Cu) (net 19))
@@
   (segment (start 67.5 92) (end 68.75 93.25) (width 0.381) (layer F.Cu) (net 31))
   (segment (start 133.291385 128.831587) (end 133.479899 129.020101) (width 1.27) (layer F.Cu) (net 32))
-  (segment (start 130.691385 126.231587) (end 131.404899 126.945101) (width 1.27) (layer F.Cu) (net 32))
-  (segment (start 130.691385 123.770062) (end 130.691385 126.231587) (width 1.27) (layer F.Cu) (net 32))
-  (segment (start 133.479899 129.020101) (end 141.791385 123.770062) (width 1.27) (layer F.Cu) (net 32))
   (segment (start 131.404899 126.945101) (end 133.479899 129.020101) (width 1.27) (layer F.Cu) (net 32))
   (via (at 131.5 127.25) (size 2) (drill 1.2) (layers F.Cu B.Cu) (net 32))
+  (segment (start 141.291385 124.270062) (end 133.479899 129.020101) (width 1.27) (layer F.Cu) (net 32))
+  (segment (start 131.5 127.25) (end 130.041385 123.770062) (width 1.27) (layer F.Cu) (net 32))
   (segment (start 128.190202 131.65) (end 129.520101 132.979899) (width 1.27) (layer F.Cu) (net 33))
   (segment (start 121.5 131.65) (end 128.190202 131.65) (width 1.27) (layer F.Cu) (net 33))
@@
   (segment (start 133.92 108.635) (end 133.92 112.070002) (width 0.508) (layer B.Cu) (net 45))
   (segment (start 133.92 112.070002) (end 134.099998 112.25) (width 0.508) (layer B.Cu) (net 45))
-  (segment (start 129 121.25) (end 126.558622 121.842923) (width 0.508) (layer F.Cu) (net 45))
   (segment (start 133.5 122.25) (end 129 121.25) (width 0.508) (layer F.Cu) (net 45))
   (segment (start 136.5 115.265685) (end 136.5 115.75) (width 0.508) (layer F.Cu) (net 45))
@@
   (segment (start 135.05 106.9) (end 133.95 106.9) (width 0.635) (layer B.Cu) (net 45))
   (segment (start 133.95 106.9) (end 133.92 106.93) (width 0.635) (layer B.Cu) (net 45))
-  (segment (start 125.065363 120.349664) (end 126.558622 121.842923) (width 0.635) (layer F.Cu) (net 45))
-  (segment (start 124.353795 120.349664) (end 125.065363 120.349664) (width 0.635) (layer F.Cu) (net 45))
+  (segment (start 129 121.25) (end 125.908622 121.842923) (width 0.508) (layer F.Cu) (net 45))
+  (segment (start 123.803795 120.349664) (end 125.908622 121.842923) (width 0.508) (layer F.Cu) (net 45))
   (segment (start 120.0375 140.0375) (end 120.0375 140.5) (width 0.381) (layer F.Cu) (net 46))
   (segment (start 119.22 137.95) (end 119.22 139.22) (width 0.381) (layer F.Cu) (net 46))
   (segment (start 119.22 139.22) (end 120.0375 140.0375) (width 0.381) (layer F.Cu) (net 46))
   (via (at 138.999992 115) (size 0.8) (drill 0.4) (layers F.Cu B.Cu) (net 47))
-  (segment (start 137.658622 121.842923) (end 137.658622 116.34137) (width 0.508) (layer F.Cu) (net 47))
   (segment (start 143.37429 109.34071) (end 143.37429 110.625702) (width 0.635) (layer B.Cu) (net 47))
-  (segment (start 137.658622 116.34137) (end 138.599993 115.399999) (width 0.508) (layer F.Cu) (net 47))
   (segment (start 138.184315 115) (end 138.434307 115) (width 0.508) (layer F.Cu) (net 47))
   (segment (start 143.37429 110.625702) (end 139.399991 114.600001) (width 0.635) (layer B.Cu) (net 47))
@@
   (segment (start 144.08 108.635) (end 143.37429 109.34071) (width 0.635) (layer B.Cu) (net 47))
   (segment (start 135.25 109.4325) (end 135.25 112.065685) (width 0.508) (layer F.Cu) (net 47))
+  (segment (start 137.158622 122.342923) (end 137.35 119.15) (width 0.508) (layer F.Cu) (net 47))
+  (segment (start 137.35 119.15) (end 138.999992 115) (width 0.508) (layer F.Cu) (net 47))
   (segment (start 103.25 132.752902) (end 105.209598 134.7125) (width 0.381) (layer F.Cu) (net 48))
   (segment (start 105.209598 134.7125) (end 106 134.7125) (width 0.381) (layer F.Cu) (net 48))
@@
   )
   (zone (net 2) (net_name GND) (layer F.Cu) (hatch edge 0.508)
-    (connect_pads (clearance 0.5))
+    (connect_pads (clearance 0.381))
     (min_thickness 0.254)
     (fill yes (arc_segments 32) (thermal_gap 0.508) (thermal_bridge_width 0.508))
